File: hardware/ebike/batteryman.kicad_sch (KiCad schematic)
At the start: 0 parts

Commit message: some power management planning
Other:
- note added: "Add xt60 connector for battery input"
- note added: "Implement current sensing + voltage divider to determine battery percentage"
- note added: "Use buck + ldo 48v --> 5v --> 3.3v"
Changed lines of the file:
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@@
 	(generator_version "9.0")
 	(paper "A4")
+	(text "Add xt60 connector for battery input"
+		(exclude_from_sim no)
+		(at 202.692 25.4 0)
+		(effects
+			(font
+				(size 1.27 1.27)
+			)
+		)
+	)
+	(text "Implement current sensing + voltage divider to determine battery percentage"
+		(exclude_from_sim no)
+		(at 107.696 24.384 0)
+		(effects
+			(font
+				(size 1.27 1.27)
+			)
+		)
+	)
+	(text "Use buck + ldo\n\n48v --> 5v --> 3.3v"
+		(exclude_from_sim no)
+		(at 32.004 25.146 0)
+		(effects
+			(font
+				(size 1.27 1.27)
+			)
+		)
+	)
 )
