File: hardware/ebike/ebike.kicad_sch (KiCad schematic)
At the start: 19 parts, among them U1 STM32G431CBTx, Y1 ABLS-8MHZ-B2-T

Commit message: minor fixes
Changed lines of the file:
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@@
-	(wire
-		(pts
-			(xy 181.61 86.36) (xy 181.61 90.17)
-		)
-		(stroke
-			(width 0)
-			(type default)
-		)
-	)
 	(wire
 		(pts
@@
 	(global_label "BuzzerPWM"
 		(shape output)
-		(at 181.61 90.17 0)
+		(at 181.61 86.36 0)
 		(fields_autoplaced yes)
 		(effects
@@
 		)
 		(property "Intersheetrefs" "${INTERSHEET_REFS}"
-			(at 195.118 90.17 0)
-			(effects
-				(font
+			(at 195.118 86.36 0)
+			(effects
+				(font

Commit message: started working on footprint assignment
Parts:
- C4: value 4.7u -> 2.2u
Other:
- note added: "Is this zener diode placement correct?"
Changed lines of the file:
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@@
 	(generator_version "9.0")
 	(paper "A4")
+	(text "Is this zener diode placement correct?"
+		(exclude_from_sim no)
+		(at 223.012 62.484 0)
+		(effects
+			(font
+				(size 1.27 1.27)
+			)
+		)
+	)
 	(text "PB6-TX, PB7-RX"
 		(exclude_from_sim no)
@@
 			)
 		)
-		(property "Datasheet" "~"
+		(property "Datasheet" "https://www.digikey.com/en/products/detail/kemet/C0805C104KMREC7210/8645300"
 			(at 210.82 69.85 0)
 			(effects
@@
 			)
 		)
-		(property "Datasheet" "~"
+		(property "Datasheet" "https://www.digikey.com/en/products/detail/kemet/C0805C104KMREC7210/8645300"
 			(at 119.38 43.18 0)
 			(effects
@@
 			)
 		)
-		(property "Datasheet" "~"
+		(property "Datasheet" "https://www.digikey.com/en/products/detail/kemet/C0805C104KMREC7210/8645300"
 			(at 127 43.18 0)
 			(effects
@@
 			)
 		)
-		(property "Datasheet" "~"
+		(property "Datasheet" "https://www.digikey.com/en/products/detail/kemet/C0805C104KMREC7210/8645300"
 			(at 107.95 60.96 0)
 			(effects
@@
 			)
 		)
-		(property "Datasheet" "~"
+		(property "Datasheet" "https://www.digikey.com/en/products/detail/kemet/C0805C104KMREC7210/8645300"
 			(at 111.76 43.18 0)
 			(effects
@@
 			)
 		)
-		(property "Value" "4.7u"
+		(property "Value" "2.2u"
 			(at 135.128 45.72 0)
 			(effects
@@
 			)
 		)
-		(property "Datasheet" "~"
+		(property "Datasheet" ""
 			(at 134.62 43.18 0)
 			(effects
