File: hardware/ebike/power.kicad_sch (KiCad schematic)
At the start: 52 parts, among them IC1 DRV8302, J1 Screw_Terminal_01x02, Q1 TC2117-3.3VEBTR, SW1 SW_SPDT, SW2 SW_SPDT

Commit message: started working on footprint assignment
Parts:
- C17: value 4.7u -> 2.2u
Changed lines of the file:
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@@
 			)
 		)
-		(property "Datasheet" "~"
+		(property "Datasheet" "https://www.digikey.com/en/products/detail/kemet/C0805C104KMREC7210/8645300"
 			(at 254 119.38 0)
 			(effects
@@
 			)
 		)
-		(property "Value" "4.7u"
+		(property "Value" "2.2u"
 			(at 164.338 45.72 90)
 			(effects
@@
 			)
 		)
-		(property "Datasheet" "~"
+		(property "Datasheet" ""
 			(at 158.75 46.99 0)
 			(effects
@@
 			)
 		)
-		(property "Datasheet" "~"
+		(property "Datasheet" "https://www.digikey.com/en/products/detail/kemet/C0805C104KMREC7210/8645300"
 			(at 154.94 123.19 0)
 			(effects
@@
 			)
 		)
-		(property "Datasheet" "~"
+		(property "Datasheet" "https://www.digikey.com/en/products/detail/kemet/C0805C104KMREC7210/8645300"
 			(at 154.94 97.79 0)
 			(effects
@@
 			)
 		)
-		(property "Datasheet" "~"
+		(property "Datasheet" "https://www.digikey.com/en/products/detail/kemet/C0805C104KMREC7210/8645300"
 			(at 260.35 119.38 0)
 			(effects
@@
 			)
 		)
-		(property "Datasheet" "~"
+		(property "Datasheet" "https://www.digikey.com/en/products/detail/kemet/C0805C104KMREC7210/8645300"
 			(at 264.16 50.8 0)
 			(effects
@@
 			)
 		)
-		(property "Datasheet" "~"
+		(property "Datasheet" "https://www.digikey.com/en/products/detail/kemet/C0805C104KMREC7210/8645300"
 			(at 154.94 72.39 0)
 			(effects
@@
 			)
 		)
-		(property "Datasheet" "~"
+		(property "Datasheet" "https://www.digikey.com/en/products/detail/kemet/C0805C104KMREC7210/8645300"
 			(at 154.94 55.88 0)
 			(effects
@@
 			)
 		)
-		(property "Datasheet" "https://ww1.microchip.com/downloads/aemDocuments/documents/APID/ProductDocuments/DataSheets/21665D.pdf"
+		(property "Datasheet" "https://www.digikey.com/en/products/detail/microchip-technology/TC2117-3-3VDBTR/443726"
 			(at 246.38 49.53 0)
 			(effects
@@
 			)
 		)
-		(property "Description" ""
+		(property "Description" "https://ww1.microchip.com/downloads/aemDocuments/documents/APID/ProductDocuments/DataSheets/21665D.pdf"
 			(at 246.38 49.53 0)
 			(effects
@@
 			)
 		)
-		(property "Datasheet" "~"
+		(property "Datasheet" "https://www.digikey.com/en/products/detail/kemet/C0805C104KMREC7210/8645300"
 			(at 247.65 119.38 0)
 			(effects
@@
 			)
 		)
-		(property "Datasheet" "~"
+		(property "Datasheet" "https://www.digikey.com/en/products/detail/kemet/C0805C104KMREC7210/8645300"
 			(at 158.75 52.07 0)
 			(effects
